File: pcb/keyboard.kicad_pcb (KiCad board)
At the start: 2 copper layers, 149.2 x 105.8 mm, 48 parts

Commit message: feat(pcb): add M2 case mounting holes and clean autoroute artifacts
Place six MountingHole_2.2mm NPTH footprints (MH1-MH6) for the 3D-printed
case: top-shell posts seat on the PCB and lid towers clamp it from below.
Positions verified against the routed board so the 2.2mm drill clears all
copper by >=1.85mm, the post seat avoids solder joints, and the under-PCB
tower corridor avoids hotswap sockets, the nice!nano, JST, and the battery
pocket. Perimeter spots on the west side are fully occupied by column/row
interconnects, so two holes sit at interior four-key corners instead.

Clean up freerouting artifacts: remove two coincident duplicate vias on P3,
rewrite the RAW branch near the nano with exact junction coordinates
(removes the 0.3mm dangling overshoot), hide MH silkscreen refs, and
refill zones. DRC: 0 unconnected, 0 dangling; remaining errors are only
the two intentional power-switch pads overlapping the board edge.

Mirror the same six holes into the ergogen source of truth as a `mount`
zone with mounting_hole_npth footprints; regenerated outlines are
byte-identical, so board geometry is unchanged.

Co-Authored-By: Claude Fable 5 <noreply@anthropic.com>
Parts:
- added MH1: MountingHole_2.2mm, MountingHole:MountingHole_2.2mm, F.Cu at (8.68, -28.4)
- added MH2: MountingHole_2.2mm, MountingHole:MountingHole_2.2mm, F.Cu at (46.7, -15.4)
- added MH3: MountingHole_2.2mm, MountingHole:MountingHole_2.2mm, F.Cu at (105.2, -41.4)
- added MH4: MountingHole_2.2mm, MountingHole:MountingHole_2.2mm, F.Cu at (128.2, 2.08)
- added MH5: MountingHole_2.2mm, MountingHole:MountingHole_2.2mm, F.Cu at (65.7, 1.58)
- added MH6: MountingHole_2.2mm, MountingHole:MountingHole_2.2mm, F.Cu at (125.2, 43.1)
Routing:
- net P3: vias 4 -> 2
